File: kicad/power_system_board/power_system_board.kicad_sch (KiCad schematic)
At the start: 21 parts, among them J1 Conn_01x05_Pin, J2 Conn_01x05_Pin, J3 Conn_01x02_Pin, J4 Conn_01x02_Pin, J5 Conn_01x02_Pin, J6 Conn_01x02_Pin, J7 Conn_01x02_Pin, Q1 2N7002H, Q2 2N7002H, U1 MCP73831-2-OT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

Commit message: Need to add esp32 and fix USB latest => 08:10
Parts:
- BT1: footprint (none) -> Library:18650 cell holder - pin gap = 70mm
Other:
- moved on the sheet: J3, J7
Changed lines of the file:
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@@
 	(wire
 		(pts
-			(xy 36.83 38.1) (xy 41.91 38.1)
+			(xy 36.83 38.1) (xy 40.64 38.1)
 		)
 		(stroke
@@
 	(wire
 		(pts
-			(xy 21.59 35.56) (xy 33.02 35.56)
+			(xy 25.4 35.56) (xy 33.02 35.56)
 		)
 		(stroke
@@
 	(wire
 		(pts
-			(xy 21.59 38.1) (xy 29.21 38.1)
+			(xy 25.4 38.1) (xy 29.21 38.1)
 		)
 		(stroke
@@
 	(wire
 		(pts
-			(xy 33.02 35.56) (xy 41.91 35.56)
+			(xy 33.02 35.56) (xy 40.64 35.56)
 		)
 		(stroke
@@
 			)
 		)
-		(property "Footprint" ""
+		(property "Footprint" "Library:18650 cell holder - pin gap = 70mm"
 			(at 33.02 28.956 90)
 			(effects
@@
 	(symbol
 		(lib_id "Connector:Conn_01x02_Pin")
-		(at 46.99 38.1 180)
+		(at 45.72 38.1 180)
 		(unit 1)
 		(exclude_from_sim no)
@@
 		(fields_autoplaced yes)
 		(property "Reference" "J7"
-			(at 48.26 35.5599 0)
+			(at 46.99 35.5599 0)
 			(effects
 				(font
@@
 		)
 		(property "Value" "Conn_01x02_Pin"
-			(at 48.26 38.0999 0)
+			(at 46.99 38.0999 0)
 			(effects
 				(font
@@
 		)
 		(property "Footprint" "Connector_PinHeader_2.54mm:PinHeader_1x02_P2.54mm_Vertical"
-			(at 46.99 38.1 0)
+			(at 45.72 38.1 0)
 			(effects
 				(font
@@
 		)
 		(property "Datasheet" "~"
-			(at 46.99 38.1 0)
+			(at 45.72 38.1 0)
 			(effects
 				(font
@@
 		)
 		(property "Description" "Generic connector, single row, 01x02, script generated"
-			(at 46.99 38.1 0)
+			(at 45.72 38.1 0)
 			(effects
 				(font
@@
 	(symbol
 		(lib_id "Connector:Conn_01x02_Pin")
-		(at 16.51 35.56 0)
+		(at 20.32 35.56 0)
 		(unit 1)
 		(exclude_from_sim no)
@@
 		(fields_autoplaced yes)
 		(property "Reference" "J3"
-			(at 17.145 30.48 0)
+			(at 20.955 30.48 0)
 			(effects
 				(font
@@
 		)
 		(property "Value" "Conn_01x02_Pin"
-			(at 17.145 33.02 0)
+			(at 20.955 33.02 0)
 			(effects
 				(font
@@
 		)
 		(property "Footprint" "Connector_PinHeader_2.54mm:PinHeader_1x02_P2.54mm_Vertical"
-			(at 16.51 35.56 0)
+			(at 20.32 35.56 0)
 			(effects
 				(font
@@
 		)
 		(property "Datasheet" "~"
-			(at 16.51 35.56 0)
+			(at 20.32 35.56 0)
 			(effects
 				(font
@@
 		)
 		(property "Description" "Generic connector, single row, 01x02, script generated"
-			(at 16.51 35.56 0)
+			(at 20.32 35.56 0)
 			(effects
 				(font

Commit message: zip file from adrian
Parts:
- added J8, J9: Conn_01x16_Pin, Connector_PinHeader_2.54mm:PinHeader_1x16_P2.54mm_Vertical, symbol Connector:Conn_01x16_Pin
- added U2: ESP32-WROOM-32, RF_Module:ESP32-WROOM-32, symbol RF_Module:ESP32-WROOM-32
Connections:
- net GND: now also U2.1 (GND), U2.15 (GND), U2.38 (GND), U2.39 (GND)
- new net CLK: J9.13 (Pin_13), U2.20 (SCK/CLK)
- new net CMD: J9.14 (Pin_14), U2.19 (SCS/CMD)
- new net EN_ESP: J9.16 (Pin_16), U2.3 (EN)
- new net IO0: J8.1 (Pin_1), U2.25 (IO0)
- new net IO1: J8.2 (Pin_2), U2.35 (TXD0/IO1)
- new net IO12: J8.7 (Pin_7), U2.14 (IO12)
- new net IO13: J8.8 (Pin_8), U2.16 (IO13)
- new net IO14: J8.9 (Pin_9), U2.13 (IO14)
- new net IO15: J8.10 (Pin_10), U2.23 (IO15)
- new net IO16: J8.11 (Pin_11), U2.27 (IO16)
- new net IO17: J8.12 (Pin_12), U2.28 (IO17)
- new net IO18: J8.13 (Pin_13), U2.30 (IO18)
- new net IO19: J8.14 (Pin_14), U2.31 (IO19)
- new net IO2: J8.3 (Pin_3), U2.24 (IO2)
- new net IO21: J8.15 (Pin_15), U2.33 (IO21)
- new net IO22: J8.16 (Pin_16), U2.36 (IO22)
- new net IO23: J9.1 (Pin_1), U2.37 (IO23)
- new net IO25: J9.2 (Pin_2), U2.10 (IO25)
- new net IO26: J9.3 (Pin_3), U2.11 (IO26)
- new net IO27: J9.4 (Pin_4), U2.12 (IO27)
- new net IO3: J8.4 (Pin_4), U2.34 (RXD0/IO3)
- new net IO32: J9.5 (Pin_5), U2.8 (IO32)
- new net IO33: J9.6 (Pin_6), U2.9 (IO33)
- new net IO34: J9.7 (Pin_7), U2.6 (IO34)
- new net IO35: J9.8 (Pin_8), U2.7 (IO35)
- new net IO4: J8.5 (Pin_5), U2.26 (IO4)
- new net IO5: J8.6 (Pin_6), U2.29 (IO5)
- new net SD0: J9.9 (Pin_9), U2.21 (SDO/SD0)
- new net SD1: J9.10 (Pin_10), U2.22 (SDI/SD1)
- new net SD2: J9.11 (Pin_11), U2.17 (SHD/SD2)
- new net SD3: J9.12 (Pin_12), U2.18 (SWP/SD3)
- new net VDD_ESP: J9.15 (Pin_15), U2.2 (VDD)
- no-connect marks 0 -> 2

Commit message: Finished schema. 1,7 hours left
Parts:
- added C4, C5: 10u, Capacitor_SMD:C_0805_2012Metric, symbol Device:C
- added J10: Conn_01x06_Pin, Connector_PinHeader_2.54mm:PinHeader_1x06_P2.54mm_Vertical, symbol Connector:Conn_01x06_Pin
- added J11, J12: Conn_01x02_Pin, Connector_PinHeader_2.54mm:PinHeader_1x02_P2.54mm_Vertical, symbol Connector:Conn_01x02_Pin
- added U4: HT75xx-1-SOT89, Package_TO_SOT_SMD:SOT-89-3, symbol Regulator_Linear:HT75xx-1-SOT89
Connections:
- net +BATT: now also J10.1 (Pin_1), J11.2 (Pin_2)
- net -BATT: now also J10.2 (Pin_2)
- net GND: now also C4.2, C5.2, J10.5 (Pin_5), J10.6 (Pin_6), U4.1 (GND)
- net VBUS: now also J10.3 (Pin_3)
- net VDD_ESP renamed +3V3
- net +3V3: now also J10.4 (Pin_4), J12.1 (Pin_1)
- new net: C4.1, J11.1 (Pin_1), U4.2 (VIN)
- new net: C5.1, J12.2 (Pin_2), U4.3 (VOUT)
Other:
- moved on the sheet: J8, J9
