File: kicad/power_system_board/power_system_board.kicad_pcb (KiCad board)
At the start: 2 copper layers, 0 parts

Commit message: Checkpoint
Parts:
- added BT1: Battery_Cell, Library:18650 cell holder - pin gap = 70mm, F.Cu at (82.7, 57.7)
- added C1: 4.7u, Capacitor_SMD:C_0805_2012Metric, F.Cu at (90.1, 78.5)
- added C2: 4.7u, Capacitor_SMD:C_0805_2012Metric, F.Cu at (95.0, 75.5)
- added C3: 100n, Capacitor_SMD:C_0805_2012Metric, F.Cu at (94.0, 83.0)
- added C4: 10u, Capacitor_SMD:C_0805_2012Metric, F.Cu at (112.0, 71.5)
- added C5: 10u, Capacitor_SMD:C_0805_2012Metric, F.Cu at (108.5, 73.5)
- added D1: LED, LED_SMD:LED_0805_2012Metric, F.Cu at (95.1, 70.5)
- added J1: Conn_01x05_Pin, Connector_PinHeader_2.54mm:PinHeader_1x05_P2.54mm_Vertical, F.Cu at (144.9, 82.0)
- added J10: Conn_01x06_Pin, Connector_PinHeader_2.54mm:PinHeader_1x06_P2.54mm_Vertical, F.Cu at (124.9, 82.0)
- added J11: Conn_01x02_Pin, Connector_PinHeader_2.54mm:PinHeader_1x02_P2.54mm_Vertical, F.Cu at (111.5, 78.0)
- added J12: Conn_01x02_Pin, Connector_PinHeader_2.54mm:PinHeader_1x02_P2.54mm_Vertical, F.Cu at (116.0, 92.3)
- added J2: Conn_01x05_Pin, Connector_PinHeader_2.54mm:PinHeader_1x05_P2.54mm_Vertical, F.Cu at (155.0, 72.9)
- added J3: Conn_01x02_Pin, Connector_PinHeader_2.54mm:PinHeader_1x02_P2.54mm_Vertical, F.Cu at (89.5, 90.3)
- added J4: Conn_01x02_Pin, Connector_PinHeader_2.54mm:PinHeader_1x02_P2.54mm_Vertical, F.Cu at (81.5, 74.3)
- added J5: Conn_01x02_Pin, Connector_PinHeader_2.54mm:PinHeader_1x02_P2.54mm_Vertical, F.Cu at (103.0, 78.8)
- added J6: Conn_01x02_Pin, Connector_PinHeader_2.54mm:PinHeader_1x02_P2.54mm_Vertical, F.Cu at (98.0, 82.8)
- added J7: Conn_01x02_Pin, Connector_PinHeader_2.54mm:PinHeader_1x02_P2.54mm_Vertical, F.Cu at (91.8, 94.5)
- added J8: Conn_01x16_Pin, Connector_PinHeader_2.54mm:PinHeader_1x16_P2.54mm_Vertical, F.Cu at (151.5, 98.9)
- added J9: Conn_01x16_Pin, Connector_PinHeader_2.54mm:PinHeader_1x16_P2.54mm_Vertical, F.Cu at (89.3, 99.0)
- added Q1: 2N7002H, Package_TO_SOT_SMD:SOT-23, F.Cu at (102.5, 89.0)
- added Q2: 2N7002H, Package_TO_SOT_SMD:SOT-23, F.Cu at (102.5, 93.0)
- added R1: 2k7, Resistor_SMD:R_0805_2012Metric, F.Cu at (98.5, 93.0)
- added R2: 330, Resistor_SMD:R_0805_2012Metric, F.Cu at (90.0, 82.6)
- added R3: 2k, Resistor_SMD:R_0805_2012Metric, F.Cu at (86.1, 73.1)
- added R4: 470, Resistor_SMD:R_0805_2012Metric, F.Cu at (90.1, 70.5)
- added R5: 330m, Resistor_SMD:R_0805_2012Metric, F.Cu at (101.0, 85.0)
- added U1: MCP73831-2-OT, Package_TO_SOT_SMD:SOT-23-5, F.Cu at (90.5, 74.5)
- added U2: ESP32-WROOM-32, RF_Module:ESP32-WROOM-32, F.Cu at (120.8, 107.1)
- added U3: AP9101CK6-AYTRG1, Package_TO_SOT_SMD:SOT-23-6, F.Cu at (94.5, 87.0)
- added U4: HT75xx-1-SOT89, Package_TO_SOT_SMD:SOT-89-3, F.Cu at (117.0, 72.0)
Routing:
- net GND: track 0.00 -> 189.8 mm, vias 0 -> 3
- net Net-(BT1--): track 0.00 -> 83.2 mm, vias 0 -> 1
- net VBUS: track 0.00 -> 78.0 mm
- net +BATT: track 0.00 -> 58.3 mm, vias 0 -> 5
- net /IO35: track 0.00 -> 52.2 mm, vias 0 -> 2
- net /IO0: track 0.00 -> 48.2 mm, vias 0 -> 2
- net /SD0: track 0.00 -> 48.1 mm, vias 0 -> 2
- net /IO25: track 0.00 -> 47.3 mm, vias 0 -> 2
- net /IO33: track 0.00 -> 46.4 mm, vias 0 -> 2
- net /IO34: track 0.00 -> 45.2 mm, vias 0 -> 2
- net /IO32: track 0.00 -> 44.2 mm, vias 0 -> 2
- net /IO27: track 0.00 -> 42.4 mm, vias 0 -> 2
- net /IO26: track 0.00 -> 40.9 mm, vias 0 -> 2
- net -BATT: track 0.00 -> 37.9 mm
- net /IO13: track 0.00 -> 37.5 mm, vias 0 -> 1
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