File: kicad/power_system_board/power_system_board.kicad_pcb (KiCad board)
At the start: 2 copper layers, 30 parts, among them J1 Conn_01x05_Pin, J10 Conn_01x06_Pin, J11 Conn_01x02_Pin, J12 Conn_01x02_Pin, J2 Conn_01x05_Pin, J3 Conn_01x02_Pin, J4 Conn_01x02_Pin, J5 Conn_01x02_Pin, J6 Conn_01x02_Pin, J7 Conn_01x02_Pin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

Commit message: Checkpoint
Parts:
- moved J8 68.0 mm to (83.5, 99.0)
- moved J9 65.2 mm to (154.5, 98.0)
- moved U2 0.50 mm to (120.8, 107.6)
Routing:
- net /CMD: track 0.00 -> 93.1 mm, vias 0 -> 2
- net /CLK: track 0.00 -> 89.7 mm, vias 0 -> 2
- net /SD3: track 0.00 -> 80.4 mm, vias 0 -> 2
- net /SD2: track 0.00 -> 74.0 mm, vias 0 -> 2
- net /IO17: track 0.00 -> 70.9 mm, vias 0 -> 2
- net +3V3: track 20.8 -> 90.9 mm, vias 0 -> 2
- net /IO15: track 0.00 -> 65.4 mm, vias 0 -> 2
- net /IO18: track 0.00 -> 61.8 mm, vias 0 -> 2
- net /SD1: track 0.00 -> 53.4 mm, vias 0 -> 4
- net /IO22: track 0.00 -> 51.6 mm, vias 0 -> 2
- net /IO14: track 29.9 -> 81.3 mm, vias 0 -> 2
- net /IO21: track 0.00 -> 50.9 mm, vias 0 -> 1
- net /IO19: track 0.00 -> 45.6 mm, vias 0 -> 2
- net /IO16: track 0.00 -> 44.7 mm, vias 0 -> 3
- net /EN_ESP: track 0.00 -> 42.3 mm, vias 0 -> 2
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Other:
- board outline added: 100 x 100 mm

Commit message: Checkpoint
Routing:
- net -BATT: track 37.9 -> 46.7 mm, vias 0 -> 2
- net Net-(U3-VDD): track 3.31 -> 8.67 mm
Other:
- board text added: "+"
- board text added: "-"
- board text added: "EEE4113F Harry Papanicolaou Adrian McIntosh Nicola Watt Md Shaihan Islam"
- board text added: "Starling Weight Project"
Changed lines of the file:
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@@
 	)
 	(setup
+		(stackup
+			(layer "F.SilkS"
+				(type "Top Silk Screen")
+			)
+			(layer "F.Paste"
+				(type "Top Solder Paste")
+			)
+			(layer "F.Mask"
+				(type "Top Solder Mask")
+				(thickness 0.01)
+			)
+			(layer "F.Cu"
+				(type "copper")
+				(thickness 0.035)
+			)
+			(layer "dielectric 1"
+				(type "core")
+				(thickness 1.51)
+				(material "FR4")
+				(epsilon_r 4.5)
+				(loss_tangent 0.02)
+			)
+			(layer "B.Cu"
+				(type "copper")
+				(thickness 0.035)
+			)
+			(layer "B.Mask"
+				(type "Bottom Solder Mask")
+				(thickness 0.01)
+			)
+			(layer "B.Paste"
+				(type "Bottom Solder Paste")
+			)
+			(layer "B.SilkS"
+				(type "Bottom Silk Screen")
+			)
+			(copper_finish "None")
+			(dielectric_constraints no)
+		)
 		(pad_to_mask_clearance 0)
 		(allow_soldermask_bridges_in_footprints no)
@@
 		(tags "SOT-89-3")
 		(property "Reference" "U4"
-			(at 0 -3.5 0)
+			(at 3.5 1.5 0)
 			(layer "F.SilkS")
 			(effects
@@
 		(tags "Through hole pin header THT 1x02 2.54mm single row")
 		(property "Reference" "J3"
-			(at 0 -2.33 180)
+			(at 3 0.775 180)
 			(layer "F.SilkS")
 			(effects
@@
 	)
 	(gr_rect
-		(start 69.5 43.5)
-		(end 169.5 143.5)
+		(start 68 42.5)
+		(end 168 142.5)
 		(stroke
 			(width 0.1)
@@
 		(layer "Edge.Cuts")
 	)
+	(gr_text "EEE4113F\nHarry Papanicolaou\nAdrian McIntosh\nNicola Watt\nMd Shaihan Islam"
+		(at 144 137.5 0)
+		(layer "B.SilkS")
+		(effects
+			(font
+				(size 1 1)
+				(thickness 0.15)
+			)
+			(justify left bottom mirror)
+		)
+	)
+	(gr_text "Starling Weight Project\n"
+		(at 115.5 137.5 0)
+		(layer "B.SilkS")
+		(effects
+			(font
+				(size 1 1)
+				(thickness 0.15)
+			)
+			(justify left bottom mirror)
+		)
+	)
+	(gr_text "-"
+		(at 142.5 58.5 0)
+		(layer "F.SilkS")
+		(effects
+			(font
+				(size 1 1)
+				(thickness 0.15)
+			)
+			(justify left bottom)
+		)
+	)
+	(gr_text "+"
+		(at 94.5 58 0)
+		(layer "F.SilkS")
+		(effects
+			(font
+				(size 1 1)
+				(thickness 0.15)
+			)
+			(justify left bottom)
+		)
+	)
 	(segment
 		(start 81.5 59.9775)
@@
 	)
 	(segment
+		(start 95.5 83.5)
+		(end 95 83)
+		(width 0.25)
+		(layer "F.Cu")
+		(net 6)
+	)
+	(segment
+		(start 94.4125 89)
+		(end 95.5 89)
+		(width 0.25)
+		(layer "F.Cu")
+		(net 6)
+	)
+	(segment
 		(start 89.5 87.735)
 		(end 93.1475 87.735)
@@
 	)
 	(segment
+		(start 95.5 84.5)
+		(end 95.5 83.5)
+		(width 0.25)
+		(layer "F.Cu")
+		(net 6)
+	)
+	(segment
 		(start 95 83)
 		(end 97.775 83)
@@
 	)
 	(segment
+		(start 93.3625 87.95)
+		(end 94.4125 89)
+		(width 0.25)
+		(layer "F.Cu")
+		(net 6)
+	)
+	(segment
 		(start 98 82.775)
 		(end 99.6875 82.775)
@@
 		(net 6)
 	)
+	(via
+		(at 95.5 84.5)
+		(size 0.8)
+		(drill 0.4)
+		(layers "F.Cu" "B.Cu")
+		(net 6)
+	)
+	(via
+		(at 95.5 89)
+		(size 0.8)
+		(drill 0.4)
+		(layers "F.Cu" "B.Cu")
+		(net 6)
+	)
+	(segment
+		(start 95.5 88.5)
+		(end 95.5 84.5)
+		(width 0.25)
+		(layer "B.Cu")
+		(net 6)
+	)
+	(segment
+		(start 95.5 89)
+		(end 95.5 88.5)
+		(width 0.25)
+		(layer "B.Cu")
+		(net 6)
+	)
 	(segment
 		(start 92.6 83.5)
+		(end 91.5 83.5)
+		(width 0.25)
+		(layer "F.Cu")
+		(net 7)
+	)
+	(segment
+		(start 93.3625 87)
+		(end 91.5 87)
+		(width 0.25)
+		(layer "F.Cu")
+		(net 7)
+	)
+	(segment
+		(start 91.5 83.5)
 		(end 90 83.5)
 		(width 0.25)
@@
 		(width 0.25)
 		(layer "F.Cu")
+		(net 7)
+	)
+	(segment
+		(start 91.5 87)
+		(end 91.5 83.5)
+		(width 0.25)
+		(layer "F.Cu")

Commit message: Checkpoint
Parts:
- moved J4 2.00 mm to (81.5, 76.3)
Routing:
- net Net-(BT1-+): track 14.9 -> 16.9 mm
- net +BATT: track 58.3 -> 57.7 mm
Changed lines of the file:
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@@
 	(footprint "Connector_PinHeader_2.54mm:PinHeader_1x02_P2.54mm_Vertical"
 		(layer "F.Cu")
-		(at 81.5 74.275 180)
+		(at 81.5 76.275 180)
 		(descr "Through hole straight pin header, 1x02, 2.54mm pitch, single row")
 		(tags "Through hole pin header THT 1x02 2.54mm single row")
@@
 	)
 	(segment
-		(start 81.5 59.9775)
-		(end 83.7425 57.735)
+		(start 83.7425 71.4925)
+		(end 81.5 73.735)
 		(width 0.25)
 		(layer "F.Cu")
@@
 	)
 	(segment
-		(start 81.5 71.735)
-		(end 81.5 59.9775)
+		(start 83.7425 57.735)
+		(end 83.7425 71.4925)
 		(width 0.25)
 		(layer "F.Cu")
@@
 	)
 	(segment
-		(start 113 82)
-		(end 124.88 82)
+		(start 84.225 76.275)
+		(end 84.5 76)
 		(width 0.25)
 		(layer "F.Cu")
@@
 	)
 	(segment
-		(start 81.5 74.275)
-		(end 82.775 74.275)
+		(start 113 82)
+		(end 124.88 82)
 		(width 0.25)
 		(layer "F.Cu")
@@
 	)
 	(segment
-		(start 82.775 74.275)
-		(end 84.5 76)
+		(start 81.5 76.275)
+		(end 84.225 76.275)
 		(width 0.25)
 		(layer "F.Cu")
